File: layout/ESPDimmer.sch (KiCad schematic (older format))
At the start: 13 parts, among them P1 CONN_01X03, P2 Serial, P3 LED, P4 ProgMod, P5 DS18B20, Q1 IRLB8721, U1 TLV1117-33, U2 ESP-12E

Commit message: Removed thermometer because its readings were incorrect due to the thermal release of the voltage regulator
Parts:
- removed P5: DS18B20, TO_SOT_Packages_THT:TO-92_Inline_Narrow_Oval, symbol CONN_01X03
- removed R2: 4k7, Resistors_SMD:R_0805, symbol R_Small
- removed U1: TLV1117-33, TO_SOT_Packages_SMD:SOT-223, symbol LD1117S33CTR
- added U1: TLV1117, TO_SOT_Packages_SMD:SOT-223, symbol TLV1117
Connections:
- wire segments 49 -> 43
Other:
- moved on the sheet: C1, C2, C3, P1, P2, P3, P4, Q1, R1, U2
